File: Wiring Diagrams/1_75/kiCadWiringDiagram/kiCadWiringDiagram.kicad_pcb (KiCad board)
At the start: 2 copper layers, 191 x 36 mm, 32 parts, among them J1 ESP32, J2 Encoder Connector, J3 LED Connector, J4 Motor Connector, J5 12v Input 1, J6 12v Input 2, J7 Speaker Connector, U1 LM2596S-5, U2 MC34063AD, U3 MMC5603NJ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

Commit message: update
Parts:
- moved C4 201.3 mm to (221.0, 120.0), turned to 180 degrees
- moved C2 200.7 mm to (223.0, 95.0)
- moved U1 190.1 mm to (232.2, 107.4)
- moved C3 188.9 mm to (213.0, 95.0)
- moved F1 187.9 mm to (212.1, 104.8)
- moved F2 187.0 mm to (212.1, 102.5)
- moved L2 181.7 mm to (231.5, 119.7), turned to 90 degrees
- moved C5 179.0 mm to (204.5, 104.0), turned to -90 degrees
- moved L1 178.2 mm to (232.3, 95.0)
- moved C1 177.9 mm to (223.6, 100.5)
- moved C6 177.9 mm to (214.0, 121.0), turned to 90 degrees
- moved D3 176.3 mm to (240.5, 95.7), turned to -90 degrees
- moved R1 173.4 mm to (211.0, 121.3), turned to 90 degrees
- moved R2 168.9 mm to (207.5, 121.4), turned to 90 degrees
- moved U3 162.3 mm to (189.8, 109.2), turned to 90 degrees
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Connections:
- net Net-(D4-K) renamed +10V
- net Net-(J1-Pin_3) renamed +3V3
- C1 pad 1: Net-(D1-K) -> +12V
- C1 pad 2: Net-(D1-K) -> +12V
- C2 pad 1: Net-(D1-K) -> +12V
- C2 pad 2: Net-(D3-A) -> GND
- C3 pad 1: Net-(U1-FB) -> +5V
- C3 pad 2: Net-(D3-A) -> GND
- C4 pad 1: Net-(U1-FB) -> +5V
- C4 pad 2: Net-(D3-A) -> GND
- C5 pad 2: Net-(D3-A) -> GND
- C6 pad 2: Net-(D3-A) -> GND
- C7 pad 2: Net-(D3-A) -> GND
- D1 pad 1: Net-(D1-K) -> +12V
- D1 pad 2: Net-(D1-A) -> +12V
- D2 pad 1: Net-(D1-K) -> +12V
- D2 pad 2: Net-(D2-A) -> +12V
- D3 pad 2: Net-(D3-A) -> GND
- F1 pad 1: Net-(D1-A) -> +12V
- F1 pad 2: Net-(J6-Pin_2) -> +12V
- F2 pad 1: Net-(D2-A) -> +12V
- F2 pad 2: Net-(J5-Pin_2) -> +12V
- J1 pad 1: Net-(D3-A) -> +5V
- J1 pad 2: Net-(D3-A) -> GND
- J2 pad 2: Net-(D3-A) -> GND
- J3 pad 1: Net-(D3-A) -> +5V
- J3 pad 2: Net-(D3-A) -> GND
- J5 pad 1: Net-(D3-A) -> GND
- J5 pad 2: Net-(J5-Pin_2) -> +12V
- J6 pad 1: Net-(D3-A) -> GND
- J6 pad 2: Net-(J6-Pin_2) -> +12V
- L1 pad 1: Net-(U1-FB) -> +5V
- L2 pad 1: Net-(U1-FB) -> +5V
- R1 pad 2: Net-(D3-A) -> GND
- U1 pad 1: Net-(D1-K) -> +12V
- U1 pad 3: Net-(D3-A) -> GND
- U1 pad 4: Net-(U1-FB) -> +5V
- U1 pad 5: Net-(D3-A) -> GND
- U2 pad 2: Net-(D3-A) -> GND
- U2 pad 4: Net-(D3-A) -> GND
- U2 pad 6: Net-(U1-FB) -> +5V
- U2 pad 7: Net-(U1-FB) -> +5V
- U2 pad 8: Net-(U1-FB) -> +5V
- U3 pad A1: Net-(D3-A) -> GND
- U4 pad 14: Net-(D3-A) -> GND
- U4 pad 21: Net-(D3-A) -> GND
- U4 pad 8: Net-(D3-A) -> GND
- U4 pad 9: Net-(D3-A) -> GND
- U5 pad 11: Net-(D3-A) -> GND
- U5 pad 12: Net-(D3-A) -> GND
- U5 pad 13: Net-(D3-A) -> GND
- U5 pad 6: Net-(D3-A) -> GND
